File: freeDSP_Classic_SMD.sch (KiCad schematic (older format))
At the start: 136 parts, among them P1 RCA, P10 CONN_02X05, P11 CONN_01X06, P12 RCA, P13 RCA, P14 CONN_02X11, P2 CONN_02X03, P3 MKDSN1.5/2-5.08, P4 CONN_01X03, P5 RCA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

Commit message: General Update
* added fdsp-libraries
* redid all missing connections (update to kicad4 standard-parts)
Parts:
- C1, C16, C17, C2, C23, C26, C28, C5: symbol CP2 -> C
Connections:
- wire segments 338 -> 424

Commit message: * finished filter schematics, fixed some missing connections
* next up: power supply
Parts:
- removed C14, C22: 100p, symbol C
- removed C3, C4: 22p, symbol C
- removed C35, C36, C37, C38, C43, C44, C45, C46: C, symbol C
- removed P1, P12, P13, P5, P7, P9: RCA, symbol BNC
- removed P14: CONN_02X11, Pin_Header:Pin_Header_Straight_2x11, symbol CONN_02X11
- removed P4: CONN_01X03, Pin_Header:Pin_Header_Straight_1x03, symbol CONN_01X03
- removed R12, R5: 49K9, Resistors_SMD:R_1206, symbol R
- removed R7: 100R, Resistors_SMD:R_1206, symbol R
- removed U? (x4): NE5532, symbol NE5532
- removed X1: 12.288MHz, Crystals_SMD:Q_49U3HMS, symbol CRYSTAL
- added 6n8: 470p, symbol C
- added C? (x2): 1n5, symbol C
- added C? (x2): 3n3, symbol C
- added C?: 6n8, symbol C
- added C? (x12): 100n, symbol C
- added J? (x6): RCA_01, symbol RCA_01
- added P? (x2): STDCONN, symbol STDCONN
- added R? (x4): 1K8, Resistors_SMD:R_1206, symbol R
- added R? (x2): 1K8, symbol R
- added U? (x4): NE5532, symbol NE5532
- C1, C2, C23, C5: symbol C -> CP
- C25, C50, C51, C52: value 470p -> 6n8
- C33, C47, C48, C49: value 150p -> 1n5
- C39, C40, C41, C42: value C -> 3n3
- R10, R3: value R -> 8K
- R11, R4: value R -> 18K
- R15, R16, R24, R25, R28, R29, R30, R31: value 4K75 -> 1K8
- R17, R20, R22, R23: value R -> 1K8
- R2, R9: value R -> 7K
- R33, R34, R36, R37: value R -> 49K9
Connections:
- net labels added: MCLK_DSP, MCLK_OUT1, MCLK_OUT2, NegOpAmpSupply, PosOpAmpSupply
- net labels removed: MCLK_IN, V+, V-
- wire segments 424 -> 462
- no-connect marks 0 -> 1
Other:
- note added: "Connector 1"
- note added: "Connector 2"
- note added: "Extension Header"
- note added: "FullScale Output:\n0,9 Vrms ; 2,5Vp-p"
- note added: "NE5532-Supply Current:\nmax 16mA per IC without Load"
- note added: "TPS562200"
- note added: "should be 24,576MHz"
- note removed: "GPIO Header"
- moved on the sheet: C12, C15, C16, C17, C18, C21, C25, C30, C33, C34, C39, C40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

Commit message: Switched to relative library paths
Parts:
- D2: symbol LED -> LED-RESCUE-freeDSP_Classic_SMD
- U4: symbol 24AA256P -> 24AA256P-RESCUE-freeDSP_Classic_SMD
- U? (x12): symbol NE5532 -> NE5532-RESCUE-freeDSP_Classic_SMD
Changed lines of the file:
@@
 +3V3
 $Comp
-L LED D2
+L LED-RESCUE-freeDSP_Classic_SMD D2
 U 1 1 5525F1AF
 P 6745 10425
@@
 $EndComp
 $Comp
-L NE5532 U?
+L NE5532-RESCUE-freeDSP_Classic_SMD U?
 U 1 1 56C4A3BA
 P 13455 4950
@@
 $EndComp
 $Comp
-L NE5532 U?
+L NE5532-RESCUE-freeDSP_Classic_SMD U?
 U 2 1 56C4E202
 P 10830 4850
@@
 VOUT1
 $Comp
-L NE5532 U?
+L NE5532-RESCUE-freeDSP_Classic_SMD U?
 U 1 1 56C5307B
 P 13480 6325
@@
 $EndComp
 $Comp
-L NE5532 U?
+L NE5532-RESCUE-freeDSP_Classic_SMD U?
 U 2 1 56C53092
 P 10855 6225
@@
 VOUT2
 $Comp
-L NE5532 U?
+L NE5532-RESCUE-freeDSP_Classic_SMD U?
 U 1 1 56C58F44
 P 13480 7800
@@
 $EndComp
 $Comp
-L NE5532 U?
+L NE5532-RESCUE-freeDSP_Classic_SMD U?
 U 2 1 56C58F5B
 P 10855 7700
@@
 VOUT3
 $Comp
-L NE5532 U?
+L NE5532-RESCUE-freeDSP_Classic_SMD U?
 U 1 1 56C58FC1
 P 13505 9175
@@
 $EndComp
 $Comp
-L NE5532 U?
+L NE5532-RESCUE-freeDSP_Classic_SMD U?
 U 2 1 56C58FD8
 P 10880 9075
@@
 $EndComp
 $Comp
-L 24AA256P U4
+L 24AA256P-RESCUE-freeDSP_Classic_SMD U4
 U 1 1 5525327F
 P 2075 9475
@@
 $EndComp
 $Comp
-L NE5532 U?
+L NE5532-RESCUE-freeDSP_Classic_SMD U?
 U 1 1 576C5CA1
 P 11370 1265
@@
 $EndComp
 $Comp
-L NE5532 U?
+L NE5532-RESCUE-freeDSP_Classic_SMD U?
 U 1 1 576C5CA7
 P 13995 1165
@@
 $EndComp
 $Comp
-L NE5532 U?
+L NE5532-RESCUE-freeDSP_Classic_SMD U?
 U 1 1 576C9A4E
 P 11355 2575
@@
 $EndComp
 $Comp
-L NE5532 U?
+L NE5532-RESCUE-freeDSP_Classic_SMD U?
 U 1 1 576C9A54
 P 13980 2475
