File: Simulations/muting/KICAD/muting.sch (KiCad schematic (older format))
At the start: 37 parts, among them Q1 BSH103,215, Q10 MMBF5434, Q11 MMBF5434, Q12 MMBF5434, Q2 BSH103,215, Q3 BSH103,215, Q4 BSH103,215, Q5 BSH103,215, Q6 BSH103,215, Q7 BSH103,215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

Commit message: Updated muting schematics
Parts:
- added Q13: BSS123, symbol NMOS_GSD
- added U3: LM393, symbol LM393
Connections:
- net VCC is gone; now on net +3V3: U1.8 (VCC), U1.8 (VCC), U1.8 (VCC)
- net +3V3: now also U3.2 (_), U3.8 (V+)
- net 3.3V_SW: now also Q13.1 (G)
- net GND: now also Q13.2 (S), Q13.3 (D), U3.3 (+), U3.4 (V-)
