File: Simulations/Clock/Clock.sch (KiCad schematic (older format))
At the start: 16 parts

Commit message: part value options
Parts:
- Rs: value 200 -> 68
- renumbered C2 to C1, C1 to C2
Connections:
- wire segments 36 -> 32
Other:
- moved on the sheet: C3, Y
Changed lines of the file:
@@
 LIBS:valves
 LIBS:eigenes
-LIBS:noname-cache
 LIBS:Clock-cache
 EELAYER 26 0
@@
 P 2350 2350
 F 0 "Rs" V 2143 2350 50  0000 C CNN
-F 1 "200" V 2234 2350 50  0000 C CNN
+F 1 "68" V 2234 2350 50  0000 C CNN
 F 2 "" V 2280 2350 50  0001 C CNN
 F 3 "" H 2350 2350 50  0001 C CNN
@@
 L Crystal Y
 U 1 1 591A9F20
-P 2350 2700
-F 0 "Y" H 2350 2550 50  0000 C CNN
-F 1 "Crystal" H 2350 2877 50  0000 C CNN
-F 2 "" H 2350 2700 50  0001 C CNN
-F 3 "" H 2350 2700 50  0001 C CNN
-	1    2350 2700
+P 1925 2650
+F 0 "Y" H 1925 2500 50  0000 C CNN
+F 1 "Crystal" H 1925 2827 50  0000 C CNN
+F 2 "" H 1925 2650 50  0001 C CNN
+F 3 "" H 1925 2650 50  0001 C CNN
+	1    1925 2650
 	1    0    0    -1
 $EndComp
@@
 L C C3
 U 1 1 591AAC5C
-P 1925 2700
-F 0 "C3" V 1673 2700 50  0000 C CNN
-F 1 "27p" V 1764 2700 50  0000 C CNN
-F 2 "" H 1963 2550 50  0001 C CNN
-F 3 "" H 1925 2700 50  0001 C CNN
-	1    1925 2700
+P 2350 2650
+F 0 "C3" V 2500 2650 50  0000 C CNN
+F 1 "27p" V 2189 2650 50  0000 C CNN
+F 2 "" H 2388 2500 50  0001 C CNN
+F 3 "" H 2350 2650 50  0001 C CNN
+	1    2350 2650
 	0    1    1    0
 $EndComp
@@
 $EndComp
 $Comp
-L C C2
+L C C1
 U 1 1 591AB5A1
 P 7850 3425
-F 0 "C2" H 7965 3471 50  0000 L CNN
+F 0 "C1" H 7965 3471 50  0000 L CNN
 F 1 "100p" H 7965 3380 50  0000 L CNN
 F 2 "" H 7888 3275 50  0001 C CNN
@@
 $EndComp
 $Comp
-L C C1
+L C C2
 U 1 1 591AB707
 P 9100 3425
-F 0 "C1" H 8985 3379 50  0000 R CNN
+F 0 "C2" H 8985 3379 50  0000 R CNN
 F 1 "100p" H 8985 3470 50  0000 R CNN
 F 2 "" H 9138 3275 50  0001 C CNN
@@
 Vorschlag 2\n
 Wire Wire Line
-	1475 2750 1475 2350
+	1475 2350 1475 2750
 Wire Wire Line
 	1475 2350 2200 2350
 Wire Wire Line
+	2500 2650 3550 2650
+Wire Wire Line
 	2700 2650 2700 2750
-Connection ~ 2700 2700
-Wire Wire Line
-	1475 2700 1775 2700
-Connection ~ 1475 2700
+Connection ~ 2700 2650
+Wire Wire Line
+	1475 2650 1775 2650
+Connection ~ 1475 2650
 Connection ~ 2700 2350
 Wire Wire Line
-	3300 3450 3525 3450
-Wire Wire Line
-	3300 1600 3300 3450
-Wire Wire Line
-	3300 2000 3525 2000
-Connection ~ 3300 2000
-Wire Wire Line
-	5450 2350 5450 3050
-Wire Wire Line
-	3525 3050 3350 3050
-Wire Wire Line
-	3350 3050 3350 4000
-Wire Wire Line
-	2075 2700 2200 2700
-Wire Wire Line
-	8050 3100 7850 3100
+	3350 2950 3550 2950
+Wire Wire Line
+	3350 2950 3350 4000
+Wire Wire Line
+	2075 2650 2200 2650
+Wire Wire Line
+	7850 3100 8050 3100
 Connection ~ 7850 3100
 Wire Wire Line
@@
 	8525 1775 9100 1775
 Connection ~ 9100 2325
-Wire Wire Line
-	2500 2700 3075 2700
-Wire Wire Line
-	3075 2700 3075 2350
-Wire Wire Line
-	3075 2350 3525 2350
-Wire Wire Line
-	2500 2350 3000 2350
-Wire Wire Line
-	3000 2350 3000 2525
-Wire Wire Line
-	3000 2525 3175 2525
-Wire Wire Line
-	3175 2525 3175 2700
-Wire Wire Line
-	3175 2700 3525 2700
 Wire Wire Line
 	9100 1775 9100 2550
@@
 P 9100 2700
 F 0 "Rs" H 9170 2746 50  0000 L CNN
-F 1 "200" H 9170 2655 50  0000 L CNN
+F 1 "68" H 9170 2655 50  0000 L CNN
 F 2 "" V 9030 2700 50  0001 C CNN
 F 3 "" H 9100 2700 50  0001 C CNN
@@
 Text Notes 600  7575 0    60   ~ 0
 Für Verteilung und Vorschlag 2 stehen ein inverter und ein invertierender Schmitttrigger zum Test bereit.\nAufgrund fehlender Parameter der Kristall-Ersatzschaltung kann keine der Schaltungen simuliert werden.\nDie angegebene Dimensionierung der Bauelemente ist mit einer Schätzung behaftet und experimentel sowohl für eine Testschaltung als\nauch für das finale Layout zu überprüfen\n
+Wire Wire Line
+	2500 2350 3550 2350
+Wire Wire Line
+	3200 2650 3200 2700
+Wire Wire Line
+	3300 3250 3550 3250
+Wire Wire Line
+	3300 1600 3300 3250
+Wire Wire Line
+	3300 2050 3550 2050
+Connection ~ 3300 2050
+Wire Wire Line
+	5450 2350 5450 2950
+Wire Wire Line
+	5450 3250 5450 3450
 $EndSCHEMATC

Commit message: Updated clock schematic and added footprints
Parts:
- removed U: 74AHCU04N, symbol 74AHC1G14
- added C: 10n, Capacitors_SMD:C_1206_HandSoldering, symbol C
- added C (x2): 100n, Capacitors_SMD:C_1206_HandSoldering, symbol C
- added C: 100n, symbol C
- added R (x4): 33, Resistors_SMD:R_1206_HandSoldering, symbol R
- added U: 74AC14, SMD_Packages:SOIC-14_N, symbol 74AC14
- added unit 2 of U
- added unit 3 of U
- added unit 4 of U
- added unit 5 of U
- added unit 6 of U
- U: value Crystal_Oscillator -> ASV-24.576MHZ-EJ-T; footprint (none) -> Oscillators:Oscillator_SMD_Abracon_ASV-4pin_7.0x5.1mm_HandSoldering
Connections:
- net labels added: MCLK0, MCLK1, MCLK2, MCLK3, MCLK4
- net labels removed: MCLK0-4
- wire segments 32 -> 51
- no-connect marks 0 -> 1
Other:
- note added: "Verteilung\n"
- note added: "Vorschlag 1"
- note added: "Vorschlag 2\n\n"
- note removed: "Für Verteilung und Vorschlag 2 stehen ein inverter und ein invertierender Schmitttrigger zum Test bereit.\nAufgrund fehlender Parameter der Kristall-Ersatzschaltung kann keine der Schaltungen simuliert werden.\nDie angegebene Dimensionierung der Bauelemente ist mit einer Schätzung behaftet und experimentel sowohl für eine Testschaltung als\nauch für das finale Layout zu überprüfen\n"
- note removed: "Verteilung\n\n\n"
- note removed: "Vorschlag 1\n"
- note removed: "Vorschlag 2\n"
- moved on the sheet: C1, C2, C3, Rf, Rs, U, Y
