File: SOURCES/filter.sch (KiCad schematic (older format))
At the start: 54 parts, among them J1 RCA_01, J2 RCA_01, J3 RCA_01, J4 RCA_01

Commit message: Updated schematics and labels
Parts:
- removed C10, C8, C9: 330p, fdsp_capacitor:C_0805_HandSoldering, symbol C
- removed C11, C12, C13: 560p, fdsp_capacitor:C_0805_HandSoldering, symbol C
- removed C14, C15, C16: 10u, Capacitors_SMD:CP_Elec_4x4.5, symbol C
- removed C5, C6, C7: 100p, fdsp_capacitor:C_0805_HandSoldering, symbol C
- removed J1, J2, J3, J4: RCA_01, fdsp_connector:RCA_01_CBP-G, symbol RCA_01
- removed R10, R11, R12: 2k4, fdsp_resistor:R_0805_HandSoldering, symbol R
- removed R4, R5, R6: 2k, fdsp_resistor:R_0805_HandSoldering, symbol R
- removed R7, R8, R9: 16k, fdsp_resistor:R_0805_HandSoldering, symbol R
- removed R? (x3): 49k9, symbol R
- removed U? (x3): LME49721, symbol LM358
- added C21, C22, C23: 100p, fdsp_capacitor:C_0805_HandSoldering, symbol C
- added C25, C26, C27: 330p, fdsp_capacitor:C_0805_HandSoldering, symbol C
- added C29, C30, C31: 560p, fdsp_capacitor:C_0805_HandSoldering, symbol C
- added C33, C34, C35: 10u, Capacitors_SMD:CP_Elec_4x4.5, symbol CP
- added R13, R14, R15: 2k, fdsp_resistor:R_0805_HandSoldering, symbol R
- added R17, R18, R19: 16k, fdsp_resistor:R_0805_HandSoldering, symbol R
- added R21, R22, R23: 2k4, fdsp_resistor:R_0805_HandSoldering, symbol R
- added R25, R26, R27: 49k9, symbol R
- added unit 2 of U3
- added U4: LME49721, symbol LM358
- C32: renamed from C4; symbol C -> CP
- C36, C37: renamed from C?; value 10u -> 47u; symbol C -> CP
- R30, R33: renamed from R?; value R -> 7k
- R31, R34: renamed from R?; value R -> 8k
- R32, R35: renamed from R?; value R -> 18k
- gave numbers to parts that had none: 8
- renumbered C1 to C20, C2 to C24, C3 to C28, R1 to R12, R2 to R16, R3 to R20
Connections:
- net labels added: ADC0, ADC1, CH1_IN, CH2_IN, CH3_IN, CH4_IN, VOUT0, VOUT1, VOUT2, VOUT3
- net labels removed: ADAU_IN1, ADAU_IN2, ADAU_OUT1, ADAU_OUT2, ADAU_OUT3, ADAU_OUT4
- wire segments 116 -> 113
Other:
- moved on the sheet: U3A

Commit message: Assigned footprints
Parts:
- C20, C21, C22, C23, C24, C25, C26, C27, C28, C29, C30, C31: footprint fdsp_capacitor:C_0805_HandSoldering -> fdsp_capacitor:C_1206_HandSoldering
- C32, C33, C34, C35: footprint Capacitors_SMD:CP_Elec_4x4.5 -> fdsp_capacitor:C_Radial_D5_L11_P2
- C36, C37: footprint (none) -> fdsp_capacitor:C_Radial_D5_L11_P2
- J1, J2: footprint (none) -> fdsp_connector:RCA_RCJ-01x
- P8, P9: footprint (none) -> fdsp_pinheader:Pin_Header_Straight_2x03
- R12, R13, R14, R15, R16, R17, R18, R19, R20, R21, R22, R23: footprint fdsp_resistor:R_0805_HandSoldering -> fdsp_resistor:R_1206_HandSoldering
- R24, R25, R26, R27, R28, R29, R30, R31, R32, R33, R34, R35: footprint (none) -> fdsp_resistor:R_1206_HandSoldering
- U3, U4: footprint (none) -> fdsp_housing_new:SOIC-8_3.9x4.9mm_Pitch1.27mm

Commit message: updated schematic + bom + pcb start
Parts:
- added C36, C37: 10u, fdsp_capacitor:C_Radial_D5_L11_P2, symbol CP
- added C40, C41: 100n, fdsp_capacitor:C_1206_HandSoldering, symbol C
- renumbered C36 to C38, C37 to C39
Connections:
- wire segments 113 -> 123
Changed lines of the file:
@@
 EESchema Schematic File Version 2
+LIBS:freeDSP_Classic_SMD-rescue
 LIBS:fdsp_device_new
 LIBS:fdsp_digital_new
@@
 $EndComp
 $Comp
-L CP C36
+L CP C38
 U 1 1 592C428E
 P 9000 1800
-F 0 "C36" H 9025 1900 50  0000 L CNN
+F 0 "C38" H 9025 1900 50  0000 L CNN
 F 1 "47u" H 9025 1700 50  0000 L CNN
 F 2 "fdsp_capacitor:C_Radial_D5_L11_P2" H 9038 1650 50  0001 C CNN
@@
 $EndComp
 $Comp
-L CP C37
+L CP C39
 U 1 1 592C64BF
 P 9100 4100
-F 0 "C37" H 9125 4200 50  0000 L CNN
+F 0 "C39" H 9125 4200 50  0000 L CNN
 F 1 "47u" H 9125 4000 50  0000 L CNN
 F 2 "fdsp_capacitor:C_Radial_D5_L11_P2" H 9138 3950 50  0001 C CNN
@@
 Wire Wire Line
 	1550 5150 1250 5150
+$Comp
+L GND #PWR065
+U 1 1 592EE586
+P 8450 6200
+F 0 "#PWR065" H 8450 5950 50  0001 C CNN
+F 1 "GND" H 8450 6050 50  0000 C CNN
+F 2 "" H 8450 6200 60  0000 C CNN
+F 3 "" H 8450 6200 60  0000 C CNN
+	1    8450 6200
+	1    0    0    -1
+$EndComp
+$Comp
+L CP C36
+U 1 1 592EE7F4
+P 8450 5900
+F 0 "C36" H 8475 6000 50  0000 L CNN
+F 1 "10u" H 8475 5800 50  0000 L CNN
+F 2 "fdsp_capacitor:C_Radial_D5_L11_P2" H 8488 5750 50  0001 C CNN
+F 3 "" H 8450 5900 50  0000 C CNN
+	1    8450 5900
+	1    0    0    -1
+$EndComp
+$Comp
+L CP C37
+U 1 1 592EE981
+P 8750 5900
+F 0 "C37" H 8775 6000 50  0000 L CNN
+F 1 "10u" H 8775 5800 50  0000 L CNN
+F 2 "fdsp_capacitor:C_Radial_D5_L11_P2" H 8788 5750 50  0001 C CNN
+F 3 "" H 8750 5900 50  0000 C CNN
+	1    8750 5900
+	1    0    0    -1
+$EndComp
+$Comp
+L +3V3 #PWR066
+U 1 1 592EEA39
+P 8450 5600
+F 0 "#PWR066" H 8450 5450 50  0001 C CNN
+F 1 "+3V3" H 8450 5740 50  0000 C CNN
+F 2 "" H 8450 5600 50  0000 C CNN
+F 3 "" H 8450 5600 50  0000 C CNN
+	1    8450 5600
+	1    0    0    -1
+$EndComp
+$Comp
+L C C40
+U 1 1 592EED51
+P 9150 5900
+F 0 "C40" H 9175 6000 50  0000 L CNN
+F 1 "100n" H 9175 5800 50  0000 L CNN
+F 2 "fdsp_capacitor:C_1206_HandSoldering" H 9188 5750 50  0001 C CNN
+F 3 "" H 9150 5900 50  0000 C CNN
+	1    9150 5900
+	1    0    0    -1
+$EndComp
+$Comp
+L C C41
+U 1 1 592EEF8E
+P 9450 5900
+F 0 "C41" H 9475 6000 50  0000 L CNN
+F 1 "100n" H 9475 5800 50  0000 L CNN
+F 2 "fdsp_capacitor:C_1206_HandSoldering" H 9488 5750 50  0001 C CNN
+F 3 "" H 9450 5900 50  0000 C CNN
+	1    9450 5900
+	1    0    0    -1
+$EndComp
+Wire Wire Line
+	8450 5600 8450 5750
+Wire Wire Line
+	8450 5700 9450 5700
+Wire Wire Line
+	9450 5700 9450 5750
+Wire Wire Line
+	9450 6050 9450 6100
+Wire Wire Line
+	9450 6100 8450 6100
+Wire Wire Line
+	8450 6050 8450 6200
+Connection ~ 8450 6100
+Wire Wire Line
+	8750 6050 8750 6100
+Connection ~ 8750 6100
+Wire Wire Line
+	9150 6050 9150 6100
+Connection ~ 9150 6100
+Wire Wire Line
+	9150 5750 9150 5700
+Connection ~ 9150 5700
+Wire Wire Line
+	8750 5750 8750 5700
+Connection ~ 8750 5700
+Connection ~ 8450 5700
 $EndSCHEMATC
