File: SOURCES/freeDSP_Classic_SMD.sch (KiCad schematic (older format))
At the start: 144 parts, among them P10 CONN_02X05, P11 CONN_01X06, P2 CONN_02X03, P3 MKDSN1.5/2-5.08, P6 CONN_02X03, P8 CONN_01X03, Q1 FZT751TA, Q2 2N7000, Q3 2N7000, Q4 2N7000, Q5 2N7000, SW1 SW_PUSH, U1 LD1117S33TR, U2 ADAU1701, U4 24AA256SN

Commit message: Updated folder structure
Parts:
- D2: symbol LED -> LED-RESCUE-freeDSP_Classic_SMD
- U4: symbol 24AA256P -> 24AA256P-RESCUE-freeDSP_Classic_SMD
- U? (x12): symbol NE5532 -> NE5532-RESCUE-freeDSP_Classic_SMD
- gave numbers to parts that had none: 31

Commit message: Updated schematics and added subcircuits to main sheet
Parts:
- removed 6n8: 470p, symbol C
- removed C12, C18, C21, C30, C34, C53, C54, C55, C56, C57, C58, C8: 4u7, symbol C
- removed C14, C22, C3, C35, C36, C37, C38, C4, C46, C59, C60, C61: 100n, symbol C
- removed C15: 100n, Resistors_SMD:R_1206, symbol C
- removed C16: 47u, symbol C
- removed C17: 100u, symbol C
- removed C25, C43, C50, C51, C52: 6n8, symbol C
- removed C33, C44, C45, C47, C48, C49: 1n5, symbol C
- removed C39, C40, C41, C42, C62, C63: 3n3, symbol C
- removed D1, D5: FM5818, Diodes_SMD_2:DO214AC, symbol DIODESCH
- removed D2: LED, KOMA Parts:LED-3MM, symbol LED-RESCUE-freeDSP_Classic_SMD
- removed J1, J2, J3, J4, J5, J6: RCA_01, symbol RCA_01
- removed P2, P6: CONN_02X03, Pin_Header:Pin_Header_Straight_2x03, symbol CONN_02X03
- removed P3: MKDSN1.5/2-5.08, symbol CONN_01X02
- removed R10, R3: 8K, Resistors_SMD:R_1206, symbol R
- removed R11, R4: 18K, Resistors_SMD:R_1206, symbol R
- removed R12, R15, R16, R24, R25, R28, R29, R30, R31, R38, R5, R7: 1K8, Resistors_SMD:R_1206, symbol R
- removed R17, R20, R22, R23, R39, R40: 1K8, symbol R
- removed R2, R9: 7K, Resistors_SMD:R_1206, symbol R
- removed R33, R34, R36, R37: 49K9, symbol R
- removed R8: 100R, Resistors_SMD:R_1206, symbol R
- removed U1: LD1117S33TR, SMD_Packages:SOT-223, symbol LD1117X33
- removed U? (x12): NE5532, symbol NE5532-RESCUE-freeDSP_Classic_SMD
- added P? (x2): STDCONN, symbol STDCONN
- R19, R21: value R -> 10k
- U2: footprint Housing_QFP:LQFP-48_7x7mm_Pitch0.5mm -> fdsp_housing_new:LQFP-48_7x7mm_Pitch0.5mm
- U4: footprint Housing_SOIC:SOIC-8_3.9x4.9mm_Pitch1.27mm -> fdsp_housing_new:SOIC-8_3.9x4.9mm_Pitch1.27mm; symbol 24AA256P-RESCUE-freeDSP_Classic_SMD -> 24AA256P
Connections:
- net labels added: MCLK_OUT3, MCLK_OUT4
- net labels removed: IN_BCLK, IN_LRCLK, NegOpAmpSupply, PosOpAmpSupply, SDATA_IN
- wire segments 462 -> 202
Other:
- note added: "Connector 3"
- note added: "Connector 4"
- note removed: "AC Coupling"
- note removed: "Analog Inputs"
- note removed: "Analog Output Filter"
- note removed: "FullScale Output:\n0,9 Vrms ; 2,5Vp-p"
- note removed: "Input Voltage Selector"
- note removed: "NE5532-Supply Current:\nmax 16mA per IC without Load"
- note removed: "Power Supply"
- note removed: "TPS562200"
- note removed: "should be 24,576MHz"

Commit message: Updated schematics
Parts:
- D3, D4: value FM5818 -> B140; footprint Diodes_SMD_2:DO214AC -> fdsp_diode:SMA; symbol DIODESCH -> D_Schottky
- P10: footprint Pin_Header:Pin_Header_Angled_2x05 -> fdsp_pinheader:Pin_Header_Angled_2x05
Connections:
- wire segments 202 -> 204
Changed lines of the file:
@@
 F 0 "P10" H 5125 5925 50  0000 C CNN
 F 1 "CONN_02X05" H 5125 5325 50  0000 C CNN
-F 2 "Pin_Header:Pin_Header_Angled_2x05" H 5125 4425 60  0001 C CNN
+F 2 "fdsp_pinheader:Pin_Header_Angled_2x05" H 5125 4425 60  0001 C CNN
 F 3 "" H 5125 4425 60  0000 C CNN
 	1    5125 5625
@@
 Text Label 4750 5525 2    59   ~ 0
 SDA
-$Comp
-L DIODESCH D4
-U 1 1 55259681
-P 5500 5325
-F 0 "D4" H 5500 5425 40  0000 C CNN
-F 1 "FM5818" H 5500 5225 40  0000 C CNN
-F 2 "Diodes_SMD_2:DO214AC" H 5500 5325 60  0001 C CNN
-F 3 "" H 5500 5325 60  0000 C CNN
-	1    5500 5325
-	0    -1   -1   0
-$EndComp
 Text Label 5675 5525 0    59   ~ 0
 +5V_USBI
@@
 +5V
 $Comp
-L DIODESCH D3
+L D_Schottky D3
 U 1 1 55266EFC
 P 2700 5175
 F 0 "D3" H 2700 5275 40  0000 C CNN
-F 1 "FM5818" H 2700 5075 40  0000 C CNN
-F 2 "Diodes_SMD_2:DO214AC" H 2700 5175 60  0001 C CNN
+F 1 "B140" H 2700 5075 40  0000 C CNN
+F 2 "fdsp_diode:SMA" H 2700 5175 60  0001 C CNN
 F 3 "" H 2700 5175 60  0000 C CNN
 	1    2700 5175
-	0    -1   -1   0
+	0    1    1    0
 $EndComp
 Text Label 2550 4975 2    59   ~ 0
@@
 	5675 5625 5375 5625
 Wire Wire Line
-	5500 5050 5500 5125
+	5500 5050 5500 5175
 Wire Wire Line
 	5525 5875 5525 5825
@@
 	2575 5450 2825 5450
 Wire Wire Line
-	2700 5375 2700 5450
+	2700 5325 2700 5450
 Connection ~ 2700 5450
 Wire Wire Line
@@
 Wire Wire Line
 	2775 9575 2775 9475
+$Comp
+L D_Schottky D4
+U 1 1 55259681
+P 5500 5325
+F 0 "D4" H 5500 5425 40  0000 C CNN
+F 1 "B140" H 5500 5225 40  0000 C CNN
+F 2 "fdsp_diode:SMA" H 5500 5325 60  0001 C CNN
+F 3 "" H 5500 5325 60  0000 C CNN
+	1    5500 5325
+	0    1    1    0
+$EndComp
+Wire Wire Line
+	5500 5475 5500 5525
+Wire Wire Line
+	2700 4975 2700 5025
 $EndSCHEMATC

Commit message: marker
Connections:
- wire segments 204 -> 200
Other:
- moved on the sheet: C31, D3, P11, P8, R14, R19, R21, R26, R27, R32, R35, U4

Commit message: Updated schematics and labels
Parts:
- removed P1, P? (x2): STDCONN, symbol STDCONN
- removed Q2, Q3, Q4, Q5: 2N7000, Housings_SOT-23_SOT-143_TSOT-6.pretty:SOT-23, symbol MOSFET_N
- added P5, P6, P7: STDCONN, symbol STDCONN
- added Q1, Q2, Q3, Q4: BSS123, fdsp_housing_new:SOT-23, symbol NMOS_GSD
- renumbered C32 to C1, C11 to C10, C13 to C11, C28 to C12, C29 to C13, C23 to C14, C26 to C15, C24 to C16, C27 to C17, C19 to C18, C20 to C19, C1 to C2, C6 to C3, C10 to C4, C31 to C5, C5 to C6, C9 to C7, C2 to C8, C7 to C9, D3 to D1, D4 to D2, P8 to P1, P11 to P2, P10 to P3, Q1 to Q5, R13 to R1, R18 to R10, R6 to R11, R14 to R2, R26 to R3, R27 to R4, R32 to R5, R35 to R6, R1 to R7, R19 to R8, R21 to R9, U4 to U1
Connections:
- net labels added: +12V, MCLK0, MCLK1, MCLK2, MCLK3, MCLK4
- net labels removed: +5V_USBI, MCLK_DSP, MCLK_OUT1, MCLK_OUT2, MCLK_OUT3, MCLK_OUT4, MP4, MP5, WB
- wire segments 200 -> 178
- no-connect marks 1 -> 9
Other:
- moved on the sheet: C1, C10, C11, C12, C13, C14, C15, C16, C17, C18, C19, C2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

Commit message: Assigned footprints
Parts:
- C1, C10, C11, C13, C16, C17, C3, C4, C5, C7, C9: footprint Resistors_SMD:R_1206 -> fdsp_capacitor:C_1206_HandSoldering
- C12, C14, C15, C18, C19, C2, C6, C8: footprint (none) -> fdsp_capacitor:C_1206_HandSoldering
- D1, D2: value B140 -> B150
- P1: footprint Pin_Header:Pin_Header_Straight_1x03 -> fdsp_pinheader:Pin_Header_Straight_1x03
- P2: footprint Pin_Header:Pin_Header_Angled_1x06 -> fdsp_pinheader:Pin_Header_Straight_1x06
- P3: footprint fdsp_pinheader:Pin_Header_Angled_2x05 -> fdsp_connector:IDC_Header_Straight_10pins
- P4, P5, P6, P7: footprint (none) -> fdsp_connector:IDC_Header_Straight_16pins
- Q1, Q2, Q3, Q4: footprint fdsp_housing_new:SOT-23 -> fdsp_housing_new:SOT-23_Handsoldering
- Q5: footprint SMD_Packages:SOT-223 -> fdsp_housing_new:SOT-223
- R1, R10, R11, R2, R3, R4, R5, R6, R7, R8, R9: footprint Resistors_SMD:R_1206 -> fdsp_resistor:R_1206_HandSoldering
- SW1: footprint (none) -> fdsp_housing_new:SW_PUSH_6mm
Connections:
- net +3V3: now also U2.38 (PLL_MODE0)
- net GND: no longer U2.38 (PLL_MODE0)

Commit message: updated schematic + bom + pcb start
Parts:
- U1: renamed from U2; symbol ADAU1701 -> ADAU1701-RESCUE-freeDSP_Classic_SMD
- renumbered C11 to C10, C5 to C11, C6 to C5, C7 to C6, C8 to C7, C9 to C8, C10 to C9, P2 to P1, P1 to P2, R9 to R10, R3 to R2, R4 to R3, R5 to R4, R6 to R5, R7 to R6, R2 to R7, R10 to R8, R8 to R9, U1 to U2
Other:
- moved on the sheet: C11, P2, P4, P5, P6, P7, R10, R7, R9, U2

Commit message: layout finished
Parts:
- C14, C2, C5, C7: footprint fdsp_capacitor:C_1206_HandSoldering -> fdsp_capacitor:C_Radial_D5_L11_P2
Changed lines of the file:
@@
 F 0 "C2" H 3130 1010 40  0000 L CNN
 F 1 "10u" H 3136 825 40  0000 L CNN
-F 2 "fdsp_capacitor:C_1206_HandSoldering" H 3168 760 30  0001 C CNN
+F 2 "fdsp_capacitor:C_Radial_D5_L11_P2" H 3168 760 30  0001 C CNN
 F 3 "" H 3130 910 60  0000 C CNN
 	1    3130 910
@@
 F 0 "C5" H 4300 1220 40  0000 L CNN
 F 1 "10u" H 4306 1035 40  0000 L CNN
-F 2 "fdsp_capacitor:C_1206_HandSoldering" H 4338 970 30  0001 C CNN
+F 2 "fdsp_capacitor:C_Radial_D5_L11_P2" H 4338 970 30  0001 C CNN
 F 3 "" H 4300 1120 60  0000 C CNN
 	1    4300 1120
@@
 F 0 "C7" H 5070 1055 40  0000 L CNN
 F 1 "10u" H 5076 870 40  0000 L CNN
-F 2 "fdsp_capacitor:C_1206_HandSoldering" H 5108 805 30  0001 C CNN
+F 2 "fdsp_capacitor:C_Radial_D5_L11_P2" H 5108 805 30  0001 C CNN
 F 3 "" H 5070 955 60  0000 C CNN
 	1    5070 955
@@
 F 0 "C14" H 6350 2935 40  0000 L CNN
 F 1 "10u" H 6356 2750 40  0000 L CNN
-F 2 "fdsp_capacitor:C_1206_HandSoldering" H 6388 2685 30  0001 C CNN
+F 2 "fdsp_capacitor:C_Radial_D5_L11_P2" H 6388 2685 30  0001 C CNN
 F 3 "" H 6350 2835 60  0000 C CNN
 	1    6350 2835
@@
 	5215 2735 5215 2835
 Connection ~ 5215 2835
+Connection ~ 5175 7450
+Connection ~ 4475 7750
 $EndSCHEMATC
