File: SOURCES/freeDSP_Classic_SMD.sch (KiCad schematic (older format))
At the start: 47 parts, among them P1 CONN_01X06, P2 CONN_01X03, P3 CONN_02X05, P4 STDCONN, P5 STDCONN, P6 STDCONN, P7 STDCONN, Q1 BSS123, Q2 BSS123, Q3 BSS123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

Commit message: some improvements
Parts:
- R11: value 475R -> 475
Changed lines of the file:
@@
 P 7870 1805
 F 0 "R11" V 7950 1805 40  0000 C CNN
-F 1 "475R" V 7877 1806 40  0000 C CNN
+F 1 "475" V 7877 1806 40  0000 C CNN
 F 2 "fdsp_resistor:R_1206_HandSoldering" V 7800 1805 30  0001 C CNN
 F 3 "" H 7870 1805 30  0000 C CNN
