File: SOURCES/freeDSP_Classic_SMD.sch (KiCad schematic (older format))
At the start: 47 parts, among them P1 CONN_01X06, P2 CONN_01X03, P3 CONN_02X05, P4 STDCONN, P5 STDCONN, P6 STDCONN, P7 STDCONN, Q1 BSS123, Q2 BSS123, Q3 BSS123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

Commit message: Modified FZT751
Parts:
- Q5: symbol PNP -> FZT751
Changed lines of the file:
@@
 $EndComp
 $Comp
-L PNP Q5
+L FZT751 Q5
 U 1 1 5523E57B
 P 3605 1010

Commit message: Moved ADAU to correct library
Parts:
- U1: symbol ADAU1701-RESCUE-freeDSP_Classic_SMD -> ADAU1701-New
Changed lines of the file:
@@
 $EndComp
 $Comp
-L ADAU1701-RESCUE-freeDSP_Classic_SMD U1
+L ADAU1701-New U1
 U 1 1 5523CECE
 P 3800 2955

Commit message: Removed duplicate ADAU
Parts:
- U1: symbol ADAU1701-New -> ADAU1701
Changed lines of the file:
@@
 EESchema Schematic File Version 2
-LIBS:freeDSP_Classic_SMD-rescue
 LIBS:fdsp_device_new
 LIBS:fdsp_digital_new
@@
 $EndComp
 $Comp
-L ADAU1701-New U1
+L ADAU1701 U1
 U 1 1 5523CECE
 P 3800 2955
