File: SOURCES/clock.sch (KiCad schematic (older format))
At the start: 8 parts

Commit message: Updated schematics
Parts:
- added FB?: 330, fdsp_capacitor:C_0805_HandSoldering, symbol FILTER
Connections:
- wire segments 24 -> 28
Changed lines of the file:
@@
 L VCC #PWR?
 U 1 1 591AED7A
-P 2550 6000
-F 0 "#PWR?" H 2550 5850 50  0001 C CNN
-F 1 "VCC" H 2567 6173 50  0000 C CNN
-F 2 "" H 2550 6000 50  0001 C CNN
-F 3 "" H 2550 6000 50  0001 C CNN
-	1    2550 6000
+P 2700 3750
+F 0 "#PWR?" H 2700 3600 50  0001 C CNN
+F 1 "VCC" H 2717 3923 50  0000 C CNN
+F 2 "" H 2700 3750 50  0001 C CNN
+F 3 "" H 2700 3750 50  0001 C CNN
+	1    2700 3750
 	1    0    0    -1
 $EndComp
@@
 F 3 "" H 5050 4900 50  0001 C CNN
 	1    5050 4900
-	1    0    0    -1
-$EndComp
-$Comp
-L VCC #PWR?
-U 1 1 592B2EA2
-P 5050 4275
-F 0 "#PWR?" H 5050 4125 50  0001 C CNN
-F 1 "VCC" H 5050 4425 50  0000 C CNN
-F 2 "" H 5050 4275 50  0001 C CNN
-F 3 "" H 5050 4275 50  0001 C CNN
-	1    5050 4275
 	1    0    0    -1
 $EndComp
@@
 	3875 4400 5050 4400
 Wire Wire Line
-	5050 4275 5050 4500
+	5050 4025 5050 4500
 Connection ~ 5050 4400
 $Comp
@@
 	2600 6000 2600 6300
 Connection ~ 2550 6000
+$Comp
+L FILTER FB?
+U 1 1 592C47A3
+P 2700 4100
+F 0 "FB?" H 2700 4250 50  0000 C CNN
+F 1 "330" H 2700 4000 50  0000 C CNN
+F 2 "fdsp_capacitor:C_0805_HandSoldering" H 2700 4100 50  0001 C CNN
+F 3 "http://www.mouser.com/ds/2/281/c31e-794748.pdf" H 2700 4100 50  0001 C CNN
+	1    2700 4100
+	0    1    1    0
+$EndComp
+Wire Wire Line
+	3150 4025 5050 4025
+Wire Wire Line
+	3150 4450 3150 4025
+Wire Wire Line
+	2550 4450 3150 4450
+Wire Wire Line
+	2550 6000 2550 4450
+Connection ~ 2700 4450
 $EndSCHEMATC

Commit message: exchanged clock driver
Parts:
- removed U: 74AC14, SMD_Packages:SOIC-14_N, symbol 74AC14
- added U?: IDT2305-1, symbol IDT2305-1
Connections:
- net labels removed: MCLK
- wire segments 28 -> 24
- no-connect marks 1 -> 0
Other:
- moved on the sheet: C, FB?, R, X?

Commit message: exchanged clock driver
Parts:
- removed U?: IDT2305-1, symbol IDT2305-1
- added U?: IDT2305NZ, symbol IDT2305NZ
Connections:
- wire segments 24 -> 19
Changed lines of the file:
@@
 	1825 3175 2375 3175
 Wire Wire Line
-	1825 2375 2400 2375
-Wire Wire Line
-	2400 2375 3475 2375
-Wire Wire Line
-	3475 2375 5025 2375
-Wire Wire Line
-	5025 2375 5500 2375
+	1825 2375 5500 2375
 Wire Wire Line
 	3475 3175 4025 3175
@@
 	1825 2375 1825 2600
 Wire Wire Line
-	1825 2900 1825 3175
-Wire Wire Line
-	1825 3175 1825 3325
+	1825 2900 1825 3325
 Connection ~ 1825 3175
 $Comp
@@
 	0    1    1    0
 $EndComp
-$Comp
-L IDT2305-1 U?
-U 1 1 592C77EA
-P 5950 2675
-F 0 "U?" H 5750 3125 60  0000 C CNN
-F 1 "IDT2305-1" H 5950 2225 60  0000 C CNN
-F 2 "" H 5950 2325 60  0001 C CNN
-F 3 "" H 5950 2325 60  0001 C CNN
-	1    5950 2675
-	1    0    0    -1
-$EndComp
 Connection ~ 3475 2375
 Wire Wire Line
@@
 Connection ~ 1825 2375
 Wire Wire Line
-	5025 3125 5025 3250
-Wire Wire Line
-	5025 3250 5025 3325
+	5025 3125 5025 3325
 Wire Wire Line
 	5025 3250 5500 3250
@@
 Connection ~ 5025 2375
 Connection ~ 5025 3250
+$Comp
+L IDT2305NZ U?
+U 1 1 592C77F5
+P 5950 2675
+F 0 "U?" H 5750 3125 60  0000 C CNN
+F 1 "IDT2305NZ" H 5950 2225 60  0000 C CNN
+F 2 "" H 5950 2325 60  0001 C CNN
+F 3 "" H 5950 2325 60  0001 C CNN
+	1    5950 2675
+	1    0    0    -1
+$EndComp
 $EndSCHEMATC

Commit message: Updated schematics and labels
Parts:
- U7: renamed from U?; footprint (none) -> fdsp_housing_new:SOIC-8_3.9x4.9mm_Pitch1.27mm
- gave numbers to parts that had none: 2
- renumbered C to C47, C to C48, R to R44, R to R45, R to R46, R to R47
Connections:
- net labels added: +3V3
- net labels removed: VCC
Changed lines of the file:
@@
 $EndDescr
 $Comp
-L GND #PWR?
+L GND #PWR096
 U 1 1 591AEBCE
 P 1825 3325
-F 0 "#PWR?" H 1825 3075 50  0001 C CNN
+F 0 "#PWR096" H 1825 3075 50  0001 C CNN
 F 1 "GND" H 1830 3152 50  0000 C CNN
 F 2 "" H 1825 3325 50  0001 C CNN
@@
 	1    0    0    -1
 $EndComp
-$Comp
-L VCC #PWR?
-U 1 1 591AED7A
-P 1825 1675
-F 0 "#PWR?" H 1825 1525 50  0001 C CNN
-F 1 "VCC" H 1842 1848 50  0000 C CNN
-F 2 "" H 1825 1675 50  0001 C CNN
-F 3 "" H 1825 1675 50  0001 C CNN
-	1    1825 1675
-	1    0    0    -1
-$EndComp
 Text Notes 2375 2150 0    60   ~ 0
 Oscillator\n
 $Comp
-L R R
+L R R45
 U 1 1 592B42C3
 P 6600 2675
-F 0 "R" V 6680 2675 50  0000 C CNN
+F 0 "R45" V 6680 2675 50  0000 C CNN
 F 1 "33" V 6600 2675 50  0000 C CNN
 F 2 "Resistors_SMD:R_1206_HandSoldering" V 6530 2675 50  0001 C CNN
@@
 $EndComp
 $Comp
-L R R
+L R R44
 U 1 1 592B48D2
 P 6600 2525
-F 0 "R" V 6680 2525 50  0000 C CNN
+F 0 "R44" V 6680 2525 50  0000 C CNN
 F 1 "33" V 6600 2525 50  0000 C CNN
 F 2 "Resistors_SMD:R_1206_HandSoldering" V 6530 2525 50  0001 C CNN
@@
 $EndComp
 $Comp
-L R R
+L R R46
 U 1 1 592B497C
 P 6600 2825
-F 0 "R" V 6680 2825 50  0000 C CNN
+F 0 "R46" V 6680 2825 50  0000 C CNN
 F 1 "33" V 6600 2825 50  0000 C CNN
 F 2 "Resistors_SMD:R_1206_HandSoldering" V 6530 2825 50  0001 C CNN
@@
 $EndComp
 $Comp
-L R R
+L R R47
 U 1 1 592B4AA9
 P 6600 2975
-F 0 "R" V 6680 2975 50  0000 C CNN
+F 0 "R47" V 6680 2975 50  0000 C CNN
 F 1 "33" V 6600 2975 50  0000 C CNN
 F 2 "Resistors_SMD:R_1206_HandSoldering" V 6530 2975 50  0001 C CNN
@@
 	0    1    1    0
 $EndComp
-Text GLabel 7050 2375 2    60   Input ~ 0
+Text GLabel 7050 2375 2    60   Output ~ 0
 MCLK0
-Text GLabel 7050 2525 2    60   Input ~ 0
+Text GLabel 7050 2525 2    60   Output ~ 0
 MCLK1
-Text GLabel 7050 2675 2    60   Input ~ 0
+Text GLabel 7050 2675 2    60   Output ~ 0
 MCLK2
-Text GLabel 7050 2825 2    60   Input ~ 0
+Text GLabel 7050 2825 2    60   Output ~ 0
 MCLK3
-Text GLabel 7050 2975 2    60   Input ~ 0
+Text GLabel 7050 2975 2    60   Output ~ 0
 MCLK4
 Text Notes 5400 2125 2    60   ~ 0
 Distribution\n
 $Comp
-L C C
+L C C47
 U 1 1 592AC6E6
 P 1825 2750
-F 0 "C" H 1850 2850 50  0000 L CNN
+F 0 "C47" H 1850 2850 50  0000 L CNN
 F 1 "10n" H 1850 2650 50  0000 L CNN
 F 2 "Capacitors_SMD:C_1206_HandSoldering" H 1863 2600 50  0001 C CNN
@@
 $EndComp
 $Comp
-L C C
+L C C48
 U 1 1 592AE807
 P 5025 2975
-F 0 "C" H 5050 3075 50  0000 L CNN
+F 0 "C48" H 5050 3075 50  0000 L CNN
 F 1 "100n" H 5050 2875 50  0000 L CNN
 F 2 "Capacitors_SMD:C_1206_HandSoldering" H 5063 2825 50  0001 C CNN
@@
 $EndComp
 $Comp
-L GND #PWR?
+L GND #PWR097
 U 1 1 592AF105
 P 5025 3325
-F 0 "#PWR?" H 5025 3075 50  0001 C CNN
+F 0 "#PWR097" H 5025 3075 50  0001 C CNN
 F 1 "GND" H 5025 3175 50  0000 C CNN
 F 2 "" H 5025 3325 50  0001 C CNN
@@
 Connection ~ 1825 3175
 $Comp
-L Crystal_Oszillator X?
+L Crystal_Oszillator X1
 U 1 1 592DBD72
 P 2925 2925
-F 0 "X?" H 2925 3375 60  0000 C CNN
+F 0 "X1" H 2925 3375 60  0000 C CNN
 F 1 "ASV-24.576MHz-EJ-T" H 2925 2475 60  0000 C CNN
 F 2 "fdsp_crystal-oscillator_new:Oscillator_SMD_Abracon_ASV-4pin_7.0x5.1mm_HandSoldering" H 2825 2825 60  0001 C CNN
@@
 	3475 2375 3475 2675
 $Comp
-L FILTER FB?
+L FILTER FB2
 U 1 1 592C47A3
 P 1825 2025
-F 0 "FB?" H 1825 2175 50  0000 C CNN
+F 0 "FB2" H 1825 2175 50  0000 C CNN
 F 1 "330" H 1825 1925 50  0000 C CNN
 F 2 "fdsp_capacitor:C_0805_HandSoldering" H 1825 2025 50  0001 C CNN
@@
 Connection ~ 5025 3250
 $Comp
-L IDT2305NZ U?
+L IDT2305NZ U7
 U 1 1 592C77F5
 P 5950 2675
-F 0 "U?" H 5750 3125 60  0000 C CNN
+F 0 "U7" H 5750 3125 60  0000 C CNN
 F 1 "IDT2305NZ" H 5950 2225 60  0000 C CNN
-F 2 "" H 5950 2325 60  0001 C CNN
+F 2 "fdsp_housing_new:SOIC-8_3.9x4.9mm_Pitch1.27mm" H 5950 2325 60  0001 C CNN
 F 3 "" H 5950 2325 60  0001 C CNN
 	1    5950 2675
 	1    0    0    -1
 $EndComp
+$Comp
+L +3V3 #PWR098
+U 1 1 592DEC27
+P 1825 1675
+F 0 "#PWR098" H 1825 1525 50  0001 C CNN
+F 1 "+3V3" H 1825 1815 50  0000 C CNN
+F 2 "" H 1825 1675 60  0000 C CNN
+F 3 "" H 1825 1675 60  0000 C CNN
+	1    1825 1675
+	1    0    0    -1
+$EndComp

Commit message: Assigned footprints
Parts:
- C47, C48: footprint Capacitors_SMD:C_1206_HandSoldering -> fdsp_capacitor:C_1206_HandSoldering
- R44, R45, R46, R47: footprint Resistors_SMD:R_1206_HandSoldering -> fdsp_resistor:R_1206_HandSoldering
Changed lines of the file:
@@
 $EndDescr
 $Comp
-L GND #PWR096
+L GND #PWR094
 U 1 1 591AEBCE
 P 1825 3325
-F 0 "#PWR096" H 1825 3075 50  0001 C CNN
+F 0 "#PWR094" H 1825 3075 50  0001 C CNN
 F 1 "GND" H 1830 3152 50  0000 C CNN
 F 2 "" H 1825 3325 50  0001 C CNN
@@
 F 0 "R45" V 6680 2675 50  0000 C CNN
 F 1 "33" V 6600 2675 50  0000 C CNN
-F 2 "Resistors_SMD:R_1206_HandSoldering" V 6530 2675 50  0001 C CNN
+F 2 "fdsp_resistor:R_1206_HandSoldering" V 6530 2675 50  0001 C CNN
 F 3 "" H 6600 2675 50  0001 C CNN
 	1    6600 2675
@@
 F 0 "R44" V 6680 2525 50  0000 C CNN
 F 1 "33" V 6600 2525 50  0000 C CNN
-F 2 "Resistors_SMD:R_1206_HandSoldering" V 6530 2525 50  0001 C CNN
+F 2 "fdsp_resistor:R_1206_HandSoldering" V 6530 2525 50  0001 C CNN
 F 3 "" H 6600 2525 50  0001 C CNN
 	1    6600 2525
@@
 F 0 "R46" V 6680 2825 50  0000 C CNN
 F 1 "33" V 6600 2825 50  0000 C CNN
-F 2 "Resistors_SMD:R_1206_HandSoldering" V 6530 2825 50  0001 C CNN
+F 2 "fdsp_resistor:R_1206_HandSoldering" V 6530 2825 50  0001 C CNN
 F 3 "" H 6600 2825 50  0001 C CNN
 	1    6600 2825
@@
 F 0 "R47" V 6680 2975 50  0000 C CNN
 F 1 "33" V 6600 2975 50  0000 C CNN
-F 2 "Resistors_SMD:R_1206_HandSoldering" V 6530 2975 50  0001 C CNN
+F 2 "fdsp_resistor:R_1206_HandSoldering" V 6530 2975 50  0001 C CNN
 F 3 "" H 6600 2975 50  0001 C CNN
 	1    6600 2975
@@
 F 0 "C47" H 1850 2850 50  0000 L CNN
 F 1 "10n" H 1850 2650 50  0000 L CNN
-F 2 "Capacitors_SMD:C_1206_HandSoldering" H 1863 2600 50  0001 C CNN
+F 2 "fdsp_capacitor:C_1206_HandSoldering" H 1863 2600 50  0001 C CNN
 F 3 "" H 1825 2750 50  0001 C CNN
 	1    1825 2750
@@
 F 0 "C48" H 5050 3075 50  0000 L CNN
 F 1 "100n" H 5050 2875 50  0000 L CNN
-F 2 "Capacitors_SMD:C_1206_HandSoldering" H 5063 2825 50  0001 C CNN
+F 2 "fdsp_capacitor:C_1206_HandSoldering" H 5063 2825 50  0001 C CNN
 F 3 "" H 5025 2975 50  0001 C CNN
 	1    5025 2975
@@
 $EndComp
 $Comp
-L GND #PWR097
+L GND #PWR095
 U 1 1 592AF105
 P 5025 3325
-F 0 "#PWR097" H 5025 3075 50  0001 C CNN
+F 0 "#PWR095" H 5025 3075 50  0001 C CNN
 F 1 "GND" H 5025 3175 50  0000 C CNN
 F 2 "" H 5025 3325 50  0001 C CNN
@@
 $EndComp
 $Comp
-L +3V3 #PWR098
+L +3V3 #PWR096
 U 1 1 592DEC27
 P 1825 1675
-F 0 "#PWR098" H 1825 1525 50  0001 C CNN
+F 0 "#PWR096" H 1825 1525 50  0001 C CNN
 F 1 "+3V3" H 1825 1815 50  0000 C CNN
 F 2 "" H 1825 1675 60  0000 C CNN

Commit message: updated schematic + bom + pcb start
Parts:
- X1: symbol Crystal_Oszillator -> Crystal_Oszillator-RESCUE-freeDSP_Classic_SMD
- renumbered C47 to C54, C48 to C55
Changed lines of the file:
@@
 EESchema Schematic File Version 2
+LIBS:freeDSP_Classic_SMD-rescue
 LIBS:fdsp_device_new
 LIBS:fdsp_digital_new
@@
 $EndDescr
 $Comp
-L GND #PWR094
+L GND #PWR098
 U 1 1 591AEBCE
 P 1825 3325
-F 0 "#PWR094" H 1825 3075 50  0001 C CNN
+F 0 "#PWR098" H 1825 3075 50  0001 C CNN
 F 1 "GND" H 1830 3152 50  0000 C CNN
 F 2 "" H 1825 3325 50  0001 C CNN
@@
 Distribution\n
 $Comp
-L C C47
+L C C54
 U 1 1 592AC6E6
 P 1825 2750
-F 0 "C47" H 1850 2850 50  0000 L CNN
+F 0 "C54" H 1850 2850 50  0000 L CNN
 F 1 "10n" H 1850 2650 50  0000 L CNN
 F 2 "fdsp_capacitor:C_1206_HandSoldering" H 1863 2600 50  0001 C CNN
@@
 $EndComp
 $Comp
-L C C48
+L C C55
 U 1 1 592AE807
 P 5025 2975
-F 0 "C48" H 5050 3075 50  0000 L CNN
+F 0 "C55" H 5050 3075 50  0000 L CNN
 F 1 "100n" H 5050 2875 50  0000 L CNN
 F 2 "fdsp_capacitor:C_1206_HandSoldering" H 5063 2825 50  0001 C CNN
@@
 $EndComp
 $Comp
-L GND #PWR095
+L GND #PWR099
 U 1 1 592AF105
 P 5025 3325
-F 0 "#PWR095" H 5025 3075 50  0001 C CNN
+F 0 "#PWR099" H 5025 3075 50  0001 C CNN
 F 1 "GND" H 5025 3175 50  0000 C CNN
 F 2 "" H 5025 3325 50  0001 C CNN
@@
 Connection ~ 1825 3175
 $Comp
-L Crystal_Oszillator X1
+L Crystal_Oszillator-RESCUE-freeDSP_Classic_SMD X1
 U 1 1 592DBD72
 P 2925 2925
@@
 $EndComp
 $Comp
-L +3V3 #PWR096
+L +3V3 #PWR0100
 U 1 1 592DEC27
 P 1825 1675
-F 0 "#PWR096" H 1825 1525 50  0001 C CNN
+F 0 "#PWR0100" H 1825 1525 50  0001 C CNN
 F 1 "+3V3" H 1825 1815 50  0000 C CNN
 F 2 "" H 1825 1675 60  0000 C CNN

Commit message: improved layout
Parts:
- C54: value 10n -> 10u
Changed lines of the file:
@@
 P 1825 2750
 F 0 "C54" H 1850 2850 50  0000 L CNN
-F 1 "10n" H 1850 2650 50  0000 L CNN
+F 1 "10u" H 1850 2650 50  0000 L CNN
 F 2 "fdsp_capacitor:C_1206_HandSoldering" H 1863 2600 50  0001 C CNN
 F 3 "" H 1825 2750 50  0001 C CNN
