File: SOURCES/clock.sch (KiCad schematic (older format))
At the start: 9 parts, among them U7 IDT2305NZ, X1 ASV-24.576MHz-EJ-T

Commit message: changed filter resistors, clock resistors
Parts:
- R44, R45, R46, R47: value 33 -> 22
Changed lines of the file:
@@
 P 6600 2675
 F 0 "R45" V 6680 2675 50  0000 C CNN
-F 1 "33" V 6600 2675 50  0000 C CNN
+F 1 "22" V 6600 2675 50  0000 C CNN
 F 2 "fdsp_resistor:R_1206_HandSoldering" V 6530 2675 50  0001 C CNN
 F 3 "" H 6600 2675 50  0001 C CNN
@@
 P 6600 2525
 F 0 "R44" V 6680 2525 50  0000 C CNN
-F 1 "33" V 6600 2525 50  0000 C CNN
+F 1 "22" V 6600 2525 50  0000 C CNN
 F 2 "fdsp_resistor:R_1206_HandSoldering" V 6530 2525 50  0001 C CNN
 F 3 "" H 6600 2525 50  0001 C CNN
@@
 P 6600 2825
 F 0 "R46" V 6680 2825 50  0000 C CNN
-F 1 "33" V 6600 2825 50  0000 C CNN
+F 1 "22" V 6600 2825 50  0000 C CNN
 F 2 "fdsp_resistor:R_1206_HandSoldering" V 6530 2825 50  0001 C CNN
 F 3 "" H 6600 2825 50  0001 C CNN
@@
 P 6600 2975
 F 0 "R47" V 6680 2975 50  0000 C CNN
-F 1 "33" V 6600 2975 50  0000 C CNN
+F 1 "22" V 6600 2975 50  0000 C CNN
 F 2 "fdsp_resistor:R_1206_HandSoldering" V 6530 2975 50  0001 C CNN
 F 3 "" H 6600 2975 50  0001 C CNN

Commit message: Termination resistors changed to 24Ohms
Parts:
- R44, R45, R46, R47: value 22 -> 24
Changed lines of the file:
@@
 P 6600 2675
 F 0 "R45" V 6680 2675 50  0000 C CNN
-F 1 "22" V 6600 2675 50  0000 C CNN
+F 1 "24" V 6600 2675 50  0000 C CNN
 F 2 "fdsp_resistor:R_1206_HandSoldering" V 6530 2675 50  0001 C CNN
 F 3 "" H 6600 2675 50  0001 C CNN
@@
 P 6600 2525
 F 0 "R44" V 6680 2525 50  0000 C CNN
-F 1 "22" V 6600 2525 50  0000 C CNN
+F 1 "24" V 6600 2525 50  0000 C CNN
 F 2 "fdsp_resistor:R_1206_HandSoldering" V 6530 2525 50  0001 C CNN
 F 3 "" H 6600 2525 50  0001 C CNN
@@
 P 6600 2825
 F 0 "R46" V 6680 2825 50  0000 C CNN
-F 1 "22" V 6600 2825 50  0000 C CNN
+F 1 "24" V 6600 2825 50  0000 C CNN
 F 2 "fdsp_resistor:R_1206_HandSoldering" V 6530 2825 50  0001 C CNN
 F 3 "" H 6600 2825 50  0001 C CNN
@@
 P 6600 2975
 F 0 "R47" V 6680 2975 50  0000 C CNN
-F 1 "22" V 6600 2975 50  0000 C CNN
+F 1 "24" V 6600 2975 50  0000 C CNN
 F 2 "fdsp_resistor:R_1206_HandSoldering" V 6530 2975 50  0001 C CNN
 F 3 "" H 6600 2975 50  0001 C CNN

Commit message: Fixed missing rescue library
Parts:
- X1: symbol Crystal_Oszillator-RESCUE-freeDSP_Classic_SMD -> Crystal_Oszillator
Changed lines of the file:
@@
 EESchema Schematic File Version 2
-LIBS:freeDSP_Classic_SMD-rescue
 LIBS:fdsp_device_new
 LIBS:fdsp_digital_new
 LIBS:fdsp_linear_new
 LIBS:fdsp_transistor_new
+LIBS:fdsp_oscillator_new
 LIBS:fdsp_amplifier
 LIBS:fdsp_connector
@@
 LIBS:fdsp_regulator
 LIBS:fdsp_transistor
-LIBS:power
-LIBS:device
-LIBS:transistors
-LIBS:conn
-LIBS:linear
-LIBS:regul
-LIBS:74xx
-LIBS:cmos4000
-LIBS:adc-dac
-LIBS:memory
-LIBS:xilinx
-LIBS:microcontrollers
-LIBS:dsp
-LIBS:microchip
-LIBS:analog_switches
-LIBS:motorola
-LIBS:texas
-LIBS:intel
-LIBS:audio
-LIBS:interface
-LIBS:digital-audio
-LIBS:philips
-LIBS:display
-LIBS:cypress
-LIBS:siliconi
-LIBS:opto
-LIBS:atmel
-LIBS:contrib
-LIBS:valves
-LIBS:freeDSP_Classic_SMD-cache
 EELAYER 25 0
 EELAYER END
@@
 Connection ~ 1825 3175
 $Comp
-L Crystal_Oszillator-RESCUE-freeDSP_Classic_SMD X1
+L Crystal_Oszillator X1
 U 1 1 592DBD72
 P 2925 2925
