File: SOURCES/power.sch (KiCad schematic (older format))
At the start: 15 parts, among them J3 CONN_01X02

Commit message: added power led, changed via drill size
Parts:
- added D11: LED, fdsp_resistor:R_1206_HandSoldering, symbol LED
- added R48: 330, fdsp_resistor:R_1206_HandSoldering, symbol R
Connections:
- wire segments 37 -> 40
Changed lines of the file:
@@
 $EndComp
 Wire Wire Line
-	7825 4400 9450 4400
+	7825 4400 9925 4400
 Wire Wire Line
-	9450 5350 1950 5350
+	1950 5350 9925 5350
+$Comp
+L LED D11
+U 1 1 595D0A2A
+P 9925 5100
+F 0 "D11" H 9925 5200 50  0000 C CNN
+F 1 "LED" H 9925 5000 50  0000 C CNN
+F 2 "fdsp_resistor:R_1206_HandSoldering" H 9925 5100 60  0001 C CNN
+F 3 "" H 9925 5100 60  0000 C CNN
+	1    9925 5100
+	0    -1   -1   0
+$EndComp
+$Comp
+L R R48
+U 1 1 595D0AB5
+P 9925 4625
+F 0 "R48" V 10005 4625 50  0000 C CNN
+F 1 "330" V 9925 4625 50  0000 C CNN
+F 2 "fdsp_resistor:R_1206_HandSoldering" V 9855 4625 30  0001 C CNN
+F 3 "" H 9925 4625 30  0000 C CNN
+	1    9925 4625
+	1    0    0    -1
+$EndComp
+Wire Wire Line
+	9925 4400 9925 4475
+Connection ~ 9450 4400
+Wire Wire Line
+	9925 4775 9925 4900
+Wire Wire Line
+	9925 5350 9925 5300
+Connection ~ 9450 5350
 $EndSCHEMATC

Commit message: Fixed missing rescue library
Parts:
- LM1: symbol LM284x-RESCUE-freeDSP_Classic_SMD -> LM284x
Changed lines of the file:
@@
 EESchema Schematic File Version 2
-LIBS:freeDSP_Classic_SMD-rescue
 LIBS:fdsp_device_new
 LIBS:fdsp_digital_new
 LIBS:fdsp_linear_new
 LIBS:fdsp_transistor_new
+LIBS:fdsp_oscillator_new
 LIBS:fdsp_amplifier
 LIBS:fdsp_connector
@@
 LIBS:fdsp_regulator
 LIBS:fdsp_transistor
-LIBS:power
-LIBS:device
-LIBS:transistors
-LIBS:conn
-LIBS:linear
-LIBS:regul
-LIBS:74xx
-LIBS:cmos4000
-LIBS:adc-dac
-LIBS:memory
-LIBS:xilinx
-LIBS:microcontrollers
-LIBS:dsp
-LIBS:microchip
-LIBS:analog_switches
-LIBS:motorola
-LIBS:texas
-LIBS:intel
-LIBS:audio
-LIBS:interface
-LIBS:digital-audio
-LIBS:philips
-LIBS:display
-LIBS:cypress
-LIBS:siliconi
-LIBS:opto
-LIBS:atmel
-LIBS:contrib
-LIBS:valves
-LIBS:freeDSP_Classic_SMD-cache
 EELAYER 25 0
 EELAYER END
@@
 $EndDescr
 $Comp
-L LM284x-RESCUE-freeDSP_Classic_SMD LM1
+L LM284x LM1
 U 1 1 592AEAF9
 P 5350 4400
